Commit message: Added base joint state publisher.
* Added base URDF file.

File: description/ardak_description.urdf (robot description, URDF)
Before this commit: robot sam_bot, 4 links, 4 joints
Links:
- removed link base_footprint
- removed link camera_depth_frame
- removed link imu_link
- added link camera_link
- added link front_left_wheel; visual cylinder length=${wheel_width} radius=${wheel_radius}
- added link front_right_wheel; visual cylinder length=${wheel_width} radius=${wheel_radius}
- added link rear_left_wheel; visual cylinder length=${wheel_width} radius=${wheel_radius}
- added link rear_right_wheel; visual cylinder length=${wheel_width} radius=${wheel_radius}
- link base_link: geometry visual box size=${base_length} ${base_width} ${base_height}
Joints:
- removed joint base_joint
- removed joint camera_depth_joint
- removed joint camera_joint
- removed joint imu_joint
- added joint base_to_camera_joint: type fixed, parent base_link, child camera_link, origin xyz=${camera_link_xoff} ${camera_link_yoff} ${camera_link_zoff}
- added joint front_left_drive_joint: type continuous, parent base_link, child front_left_wheel, origin xyz=${-wheel_link_xoff} ${wheel_link_yoff} ${-wheel_link_zoff}
- added joint front_right_drive_joint: type continuous, parent base_link, child front_right_wheel, origin xyz=${wheel_link_xoff} ${wheel_link_yoff} ${-wheel_link_zoff}
- added joint rear_left_drive_joint: type continuous, parent base_link, child rear_left_wheel, origin xyz=${-wheel_link_xoff} ${-wheel_link_yoff} ${-wheel_link_zoff}
- added joint rear_right_drive_joint: type continuous, parent base_link, child rear_right_wheel, origin xyz=${wheel_link_xoff} ${-wheel_link_yoff} ${-wheel_link_zoff}

Commit message: Updated robot URDF description.

File: description/ardak_description.urdf (robot description, URDF)
Before this commit: robot ardak, 6 links, 5 joints
Links:
- removed link front_left_wheel
- removed link front_right_wheel
- removed link rear_left_wheel
- removed link rear_right_wheel
- added link base_footprint
Joints:
- removed joint front_left_drive_joint
- removed joint front_right_drive_joint
- removed joint rear_left_drive_joint
- removed joint rear_right_drive_joint
- added joint base_joint: type fixed, parent base_link, child base_footprint, origin xyz=0.0 0.0 ${-(wheel_radius+wheel_zoff)} rpy=0 0 0
- joint base_to_camera_joint: origin xyz=${camera_link_xoff} ${camera_link_yoff} ${camera_link_zoff} -> xyz=${base_length/2 + camera_link_xoff} ${camera_link_yoff} ${base_height/2 + camera_link_zoff}
