Commit message: Description changes for shorter 2.0 robot

File: description/ardak/model.urdf (robot description, URDF)
Before this commit: robot ardak, 17 links, 16 joints
Links:
- link center_link: geometry collision box size=0.6 0.35 0.302244; visual box size=0.6 0.35 0.302244
Joints:
- joint camera_link_joint: origin xyz=0.3236 0 0.022122000000000003 rpy=0 0 0 -> xyz=0.268 0 0.022122000000000003 rpy=0 0 0
- joint drive_wheel_front_left_joint: origin xyz=0.26397000000000004 0.258475 0.1016 rpy=0 0 0 -> xyz=0.20837 0.258475 0.1016 rpy=0 0 0
- joint drive_wheel_front_right_joint: origin xyz=0.26397000000000004 -0.258475 0.1016 rpy=0 0 0 -> xyz=0.20837 -0.258475 0.1016 rpy=0 0 0
- joint drive_wheel_rear_left_joint: origin xyz=-0.26397000000000004 0.258475 0.1016 rpy=0 0 0 -> xyz=-0.20837 0.258475 0.1016 rpy=0 0 0
- joint drive_wheel_rear_right_joint: origin xyz=-0.26397000000000004 -0.258475 0.1016 rpy=0 0 0 -> xyz=-0.20837 -0.258475 0.1016 rpy=0 0 0

Commit message: Changes to allow model to be loaded into Gazebo-Sim Fortress.

File: description/ardak/model.urdf (robot description, URDF)
Before this commit: robot ardak, 17 links, 16 joints
Links:
- link base_link: mass 0.1 -> 0.12266; geometry collision box size=0.001 0.001 0.001; visual box size=0.001 0.001 0.001
- link camera_color_frame: mass 0.1 -> 0.12266; geometry collision box size=0.001 0.001 0.001; visual box size=0.001 0.001 0.001
- link camera_color_optical_frame: mass 0.1 -> 0.12266; geometry collision box size=0.001 0.001 0.001; visual box size=0.001 0.001 0.001
- link camera_depth_frame: mass 0.1 -> 0.12266; geometry collision box size=0.001 0.001 0.001; visual box size=0.001 0.001 0.001
- link camera_depth_optical_frame: mass 0.1 -> 0.12266; geometry collision box size=0.001 0.001 0.001; visual box size=0.001 0.001 0.001
- link camera_left_ir_frame: mass 0.1 -> 0.12266; geometry collision box size=0.001 0.001 0.001; visual box size=0.001 0.001 0.001
- link camera_left_ir_optical_frame: mass 0.1 -> 0.12266; geometry collision box size=0.001 0.001 0.001; visual box size=0.001 0.001 0.001
- link camera_link: mass 0.1 -> 0.12266; geometry collision box size=0.001 0.001 0.001; visual box size=0.001 0.001 0.001
- link camera_right_ir_frame: mass 0.1 -> 0.12266; geometry collision box size=0.001 0.001 0.001; visual box size=0.001 0.001 0.001
- link camera_right_ir_optical_frame: mass 0.1 -> 0.12266; geometry collision box size=0.001 0.001 0.001; visual box size=0.001 0.001 0.001
- link center_link: geometry collision box size=0.55 0.35 0.302244; visual box size=0.55 0.35 0.302244
- link gps_sensor_link: mass 0.1 -> 0.12266; geometry collision box size=0.001 0.001 0.001; visual box size=0.001 0.001 0.001
- link imu_sensor_link: mass 0.1 -> 0.12266; geometry collision box size=0.001 0.001 0.001; visual box size=0.001 0.001 0.001
Joints:
- joint camera_link_joint: origin xyz=0.268 0 0.022122000000000003 rpy=0 0 0 -> xyz=0.24300000000000002 0 0.022122000000000003 rpy=0 0 0
- joint drive_wheel_front_left_joint: origin xyz=0.20837 0.258475 0.1016 rpy=0 0 0 -> xyz=0.18337000000000003 0.258475 0.1016 rpy=0 0 0
- joint drive_wheel_front_right_joint: origin xyz=0.20837 -0.258475 0.1016 rpy=0 0 0 -> xyz=0.18337000000000003 -0.258475 0.1016 rpy=0 0 0
- joint drive_wheel_rear_left_joint: origin xyz=-0.20837 0.258475 0.1016 rpy=0 0 0 -> xyz=-0.18337000000000003 0.258475 0.1016 rpy=0 0 0
- joint drive_wheel_rear_right_joint: origin xyz=-0.20837 -0.258475 0.1016 rpy=0 0 0 -> xyz=-0.18337000000000003 -0.258475 0.1016 rpy=0 0 0

Commit message: Moved files to prepart for Gazebo Fortress.

File: description/ardak/model.urdf (robot description, URDF)
Before this commit: robot ardak, 17 links, 16 joints
Links:
- link base_link: geometry visual box size=0.001 0.001 0.001
- link camera_color_frame: geometry visual box size=0.001 0.001 0.001
- link camera_color_optical_frame: geometry visual box size=0.001 0.001 0.001
- link camera_depth_frame: geometry visual box size=0.001 0.001 0.001
- link camera_depth_optical_frame: geometry visual box size=0.001 0.001 0.001
- link camera_left_ir_frame: geometry visual box size=0.001 0.001 0.001
- link camera_left_ir_optical_frame: geometry visual box size=0.001 0.001 0.001
- link camera_link: geometry visual box size=0.001 0.001 0.001
- link camera_right_ir_frame: geometry visual box size=0.001 0.001 0.001
- link camera_right_ir_optical_frame: geometry visual box size=0.001 0.001 0.001
- link gps_sensor_link: geometry visual box size=0.001 0.001 0.001
- link imu_sensor_link: geometry visual box size=0.001 0.001 0.001
